File: Diagrams/BioreactorPCB/BioreactorPCB.kicad_sch (KiCad schematic)
At the start: 2 parts, among them U1 ADS1115IDGS

Commit message: Pushing code for selenoid valve
Parts:
- removed U1: ADS1115IDGS, Package_SO:TSSOP-10_3x3mm_P0.5mm, symbol Analog_ADC:ADS1115IDGS
- added D1: D, symbol Device:D
- added Q1: TIP120, Package_TO_SOT_THT:TO-220-3_Vertical, symbol Transistor_BJT:TIP120
- added R1: 2.2K, symbol Device:R
- added U1: MCP23017_ML, Package_DFN_QFN:QFN-28-1EP_6x6mm_P0.65mm_EP4.25x4.25mm, symbol Interface_Expansion:MCP23017_ML
Other:
- note added: "Port Expander"
- note added: "valve stuff"
